Commit message: Continuous joints instead of large revolutes

File: vetex_support/urdf/vetex_macro.xacro (robot description, xacro)
@@ -136,31 +136,31 @@
                         <axis xyz="0 0 0" />
                 </joint>
-                <joint name="${prefix}left_front_wheel" type="revolute">
+                <joint name="${prefix}left_front_wheel" type="continuous">
                         <origin xyz="0 0.58668 0.21577" rpy="0 1 0" />
                         <parent link="${prefix}odom" />
                         <child link="${prefix}left_front_wheel" />
                         <axis xyz="0 1 0" />
-                        <limit lower="-10" upper="10" effort="0" velocity="3" />
+                        <limit effort="0" velocity="3" />
                 </joint>
-                <joint name="${prefix}left_rear_wheel" type="revolute">
+                <joint name="${prefix}left_rear_wheel" type="continuous">
                         <origin xyz="-2.0878 0.58642 0.21577" rpy="0 1 0" />
                         <parent link="${prefix}odom" />
                         <child link="${prefix}left_rear_wheel" />
                         <axis xyz="0 1 0" />
-                        <limit lower="-10" upper="10" effort="0" velocity="3" />
+                        <limit effort="0" velocity="3" />
                 </joint>
-                <joint name="${prefix}right_rear_wheel" type="revolute">
+                <joint name="${prefix}right_rear_wheel" type="continuous">
                         <origin xyz="-2.0878 -0.58668 0.21577" rpy="0 1 0" />
                         <parent link="${prefix}odom" />
                         <child link="${prefix}right_rear_wheel" />
                         <axis xyz="0 1 0" />
-                        <limit lower="-10" upper="10" effort="0" velocity="3" />
+                        <limit effort="0" velocity="3" />
                 </joint>
-                <joint name="${prefix}right_front_wheel" type="revolute">
+                <joint name="${prefix}right_front_wheel" type="continuous">
                         <origin xyz="0 -0.58642 0.21577" rpy="0 0 0" />
                         <parent link="${prefix}odom" />
                         <child link="${prefix}right_front_wheel" />
                         <axis xyz="0 1 0" />
-                        <limit lower="-10" upper="10" effort="0" velocity="3" />
+                        <limit effort="0" velocity="3" />
                 </joint>
                	<!-- end of joint list -->

Commit message: Remove /map and /odom frames

File: vetex_support/urdf/vetex_macro.xacro (robot description, xacro)
@@ -17,38 +17,4 @@
                                 <geometry>
                                         <mesh filename="package://vetex_support/meshes/collision/base_link.stl" />
-                                </geometry>
-                        </collision>
-                </link>
-                <link name="${prefix}map">
-                        <visual>
-                                <origin xyz="0 0 0" rpy="0 0 0" />
-                                <geometry>
-                                        <mesh filename="package://vetex_support/meshes/visual/map.stl" />
-                                </geometry>
-                                <material name="">
-                                        <color rgba="0.75294 0.75294 0.75294 1" />
-                                </material>
-                        </visual>
-                        <collision>
-                                <origin xyz="0 0 0" Rpy="0 0 0" />
-                                <geometry>
-                                        <mesh filename="package://vetex_support/meshes/collision/map.stl" />
-                                </geometry>
-                        </collision>
-                </link>
-                <link name="${prefix}odom">
-                        <visual>
-                                <origin xyz="0 0 0" rpy="0 0 0" />
-                                <geometry>
-                                        <mesh filename="package://vetex_support/meshes/visual/odom.stl" />
-                                </geometry>
-                                <material name="">
-                                        <color rgba="0.75294 0.75294 0.75294 1" />
-                                </material>
-                        </visual>
-                        <collision>
-                                <origin xyz="0 0 0" rpy="0 0 0" />
-                                <geometry>
-                                        <mesh filename="package://vetex_support/meshes/collision/odom.stl" />
                                 </geometry>
                         </collision>
@@ -124,19 +90,7 @@
                 <!-- end of link list -->
                 <!-- joint list -->
-                <joint name="${prefix}map" type="fixed">
-                        <origin xyz="0 0 0" rpy="0 0 0" />
-                        <parent link="${prefix}base_link" />
-                        <child link="${prefix}map" />
-                        <axis xyz="0 0 0" />
-                </joint>
-                <joint name="${prefix}odom" type="fixed">
-                        <origin xyz="0 0 0" rpy="0 0 0" />
-                        <parent link="${prefix}map" />
-                        <child link="${prefix}odom" />
-                        <axis xyz="0 0 0" />
-                </joint>
                 <joint name="${prefix}left_front_wheel" type="continuous">
                         <origin xyz="0 0.58668 0.21577" rpy="0 1 0" />
-                        <parent link="${prefix}odom" />
+                        <parent link="${prefix}base_link" />
                         <child link="${prefix}left_front_wheel" />
                         <axis xyz="0 1 0" />
@@ -145,5 +99,5 @@
                 <joint name="${prefix}left_rear_wheel" type="continuous">
                         <origin xyz="-2.0878 0.58642 0.21577" rpy="0 1 0" />
-                        <parent link="${prefix}odom" />
+                        <parent link="${prefix}base_link" />
                         <child link="${prefix}left_rear_wheel" />
                         <axis xyz="0 1 0" />
@@ -152,5 +106,5 @@
                 <joint name="${prefix}right_rear_wheel" type="continuous">
                         <origin xyz="-2.0878 -0.58668 0.21577" rpy="0 1 0" />
-                        <parent link="${prefix}odom" />
+                        <parent link="${prefix}base_link" />
                         <child link="${prefix}right_rear_wheel" />
                         <axis xyz="0 1 0" />
@@ -159,5 +113,5 @@
                 <joint name="${prefix}right_front_wheel" type="continuous">
                         <origin xyz="0 -0.58642 0.21577" rpy="0 0 0" />
-                        <parent link="${prefix}odom" />
+                        <parent link="${prefix}base_link" />
                         <child link="${prefix}right_front_wheel" />
                         <axis xyz="0 1 0" />

Commit message: Remove identity origins and consolidate colors

File: vetex_support/urdf/vetex_macro.xacro (robot description, xacro)
@@ -5,14 +5,12 @@
                 <link name="${prefix}base_link">
                         <visual>
-                                <origin rpy="0 0 0"/>
                                 <geometry>
                                         <mesh filename="package://vetex_support/meshes/visual/base_link.stl" />
                                 </geometry>
-                                <material name="">
+                                <material name="euler_gray">
                                         <color rgba="0.75294 0.75294 0.75294 1" />
                                 </material>
                         </visual>
                         <collision>
-                                <origin xyz="0 0 0" rpy="0 0 0" />
                                 <geometry>
                                         <mesh filename="package://vetex_support/meshes/collision/base_link.stl" />
@@ -22,14 +20,10 @@
                 <link name="${prefix}left_front_wheel">
                         <visual>
-                                <origin xyz="0 0 0" rpy="0 0 0" />
                                 <geometry>
                                         <mesh filename="package://vetex_support/meshes/visual/left_front_wheel.stl" />
                                 </geometry>
-                                <material name="">
-                                        <color rgba="0.75294 0.75294 0.75294 1" />
-                                </material>
+                                <material name="euler_gray"/>
                         </visual>
                         <collision>
-                                <origin xyz="0 0 0" rpy="0 0 0" />
                                 <geometry>
                                         <mesh filename="package://vetex_support/meshes/collision/left_front_wheel.stl" />
@@ -39,14 +33,10 @@
                 <link name="${prefix}left_rear_wheel">
                         <visual>
-                                <origin xyz="0 0 0" rpy="0 0 0" />
                                 <geometry>
                                         <mesh filename="package://vetex_support/meshes/visual/left_rear_wheel.stl" />
                                 </geometry>
-                                <material name="">
-                                        <color rgba="0.75294 0.75294 0.75294 1" />
-                                </material>
+                                <material name="euler_gray"/>
                         </visual>
                         <collision>
-                                <origin xyz="0 0 0" rpy="0 0 0" />
                                 <geometry>
                                         <mesh filename="package://vetex_support/meshes/collision/left_rear_wheel.stl" />
@@ -56,14 +46,12 @@
                 <link name="${prefix}right_rear_wheel">
                         <visual>
-                                <origin xyz="0 0 0" rpy="3.1415 0 0" />
+                                <origin rpy="3.1415 0 0" />
                                 <geometry>
                                         <mesh filename="package://vetex_support/meshes/visual/right_rear_wheel.stl" />
                                 </geometry>
-                                <material name="">
-                                        <color rgba="0.75294 0.75294 0.75294 1" />
-                                </material>
+                                <material name="euler_gray"/>
                                 </visual>
                         <collision>
-                                <origin xyz="0 0 0" rpy="3.1415 0 0" />
+                                <origin rpy="3.1415 0 0" />
                                 <geometry>
                                         <mesh filename="package://vetex_support/meshes/collision/right_rear_wheel.stl" />
@@ -73,14 +61,12 @@
                 <link name="${prefix}right_front_wheel">
                         <visual>
-                                <origin xyz="0 0 0" rpy="3.1415 0 0" />
+                                <origin rpy="3.1415 0 0" />
                                 <geometry>
                                         <mesh filename="package://vetex_support/meshes/visual/right_front_wheel.stl" />
                                 </geometry>
-                                <material name="">
-                                        <color rgba="0.75294 0.75294 0.75294 1" />
-                                </material>
+                                <material name="euler_gray"/>
                         </visual>
                         <collision>
-                                <origin xyz="0 0 0" rpy="3.1415 0 0" />
+                                <origin rpy="3.1415 0 0" />
                                 <geometry>
                                         <mesh filename="package://vetex_support/meshes/collision/right_front_wheel.stl" />

Commit message: Add BaseFootprint frame

File: vetex_support/urdf/vetex_macro.xacro (robot description, xacro)
@@ -18,4 +18,5 @@
                         </collision>
                 </link>
+                <link name="${prefix}base_footprint"/>
                 <link name="${prefix}left_front_wheel">
                         <visual>
@@ -76,4 +77,9 @@
                 <!-- end of link list -->
                 <!-- joint list -->
+                <joint name="${prefix}to_footprint" type="fixed">
+                    <origin xyz="-1 0 0"/>
+                    <parent link="${prefix}base_link" />
+                    <child link="${prefix}base_footprint" />
+                </joint>
                 <joint name="${prefix}left_front_wheel" type="continuous">
                         <origin xyz="0 0.58668 0.21577" rpy="0 1 0" />

Commit message: Move base_footprint to exact center

File: vetex_support/urdf/vetex_macro.xacro (robot description, xacro)
@@ -78,5 +78,5 @@
                 <!-- joint list -->
                 <joint name="${prefix}to_footprint" type="fixed">
-                    <origin xyz="-1 0 0"/>
+                    <origin xyz="-1.0439 0 0"/>
                     <parent link="${prefix}base_link" />
                     <child link="${prefix}base_footprint" />

Commit message: Euler Nav Demo with updated URDF

File: vetex_support/urdf/vetex_macro.xacro (robot description, xacro)
@@ -18,5 +18,5 @@
                         </collision>
                 </link>
-                <link name="${prefix}base_footprint"/>
+                <link name="base_footprint"/>
                 <link name="${prefix}left_front_wheel">
                         <visual>
@@ -80,5 +80,5 @@
                     <origin xyz="-1.0439 0 0"/>
                     <parent link="${prefix}base_link" />
-                    <child link="${prefix}base_footprint" />
+                    <child link="base_footprint" />
                 </joint>
                 <joint name="${prefix}left_front_wheel" type="continuous">

Commit message: Change base_footprint to vetex_base_footprint

File: vetex_support/urdf/vetex_macro.xacro (robot description, xacro)
@@ -18,5 +18,5 @@
                         </collision>
                 </link>
-                <link name="base_footprint"/>
+                <link name="${prefix}base_footprint"/>
                 <link name="${prefix}left_front_wheel">
                         <visual>
@@ -80,5 +80,5 @@
                     <origin xyz="-1.0439 0 0"/>
                     <parent link="${prefix}base_link" />
-                    <child link="base_footprint" />
+                    <child link="${prefix}base_footprint" />
                 </joint>
                 <joint name="${prefix}left_front_wheel" type="continuous">

Commit message: rotated vetex_base_footprint by 90 degrees about z in order to match the native orientation of the base

File: vetex_support/urdf/vetex_macro.xacro (robot description, xacro)
@@ -78,5 +78,5 @@
                 <!-- joint list -->
                 <joint name="${prefix}to_footprint" type="fixed">
-                    <origin xyz="-1.0439 0 0"/>
+                    <origin xyz="-1.0439 0 0" rpy="0 0 1.57"/>
                     <parent link="${prefix}base_link" />
                     <child link="${prefix}base_footprint" />
