Commit message: Added sensor models. Need to fix ASUS sensor rotation.

File: euler_support/urdf/euler.urdf (robot description, URDF)
Before this commit: robot euler, 18 links, 17 joints
Links:
- added link _bodycenter; collision box size=0.0730 0.2760 0.0720; visual mesh filename=package://euler_support/meshes/visual/asus_sensor.stl
- added link _depth_frame
- added link _rgb_frame
- added link front_sick_s300; collision mesh filename=package://euler_support/meshes/collision/sick_s300_mounting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; visual mesh filename=package://euler_support/meshes/visual/sick_s300_mounting_as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
- added link rear_sick_s300; collision mesh filename=package://euler_support/meshes/collision/sick_s300_mounting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; visual mesh filename=package://euler_support/meshes/visual/sick_s300_mounting_as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
- added link sick_nav350; collision mesh filename=package://euler_support/meshes/collision/sick_nav350.stl; visual mesh filename=package://euler_support/meshes/visual/sick_nav350.stl
Joints:
- added joint _base-bodycenter-prism-x: type fixed, parent base_link, child _bodycenter, origin xyz=0.461 0 2.103 rpy=1.5708 1.8849 0
- added joint _depth_joint: type fixed, parent _bodycenter, child _depth_frame, origin xyz=0.049 0 0 rpy=0 0 0
- added joint _rgb_joint: type fixed, parent _bodycenter, child _rgb_frame, origin xyz=0.022 0 0 rpy=0 0 0
- added joint front_sick_s300: type fixed, parent base_link, child front_sick_s300, origin xyz=0 0 0 rpy=0 0 0, axis 0 0 0
- added joint rear_sick_s300: type fixed, parent base_link, child rear_sick_s300, origin xyz=0 0 0 rpy=0 0 0, axis 0 0 0
- added joint sick_nav350: type fixed, parent base_link, child sick_nav350, origin xyz=0 0 0 rpy=0 0 0, axis 0 0 0

File: euler_support/urdf/euler_macro.xacro (robot description, xacro)
@@ -1,20 +1,22 @@
 <?xml version="1.0" ?>
 <robot xmlns:xacro="http://ros.org/wiki/xacro">
+<xacro:include filename="$(find vetex_support)/urdf/vetex_macro.xacro" />
 <xacro:include filename="$(find motoman_mh5lf_support)/urdf/mh5lf_macro.xacro" />
-<xacro:include filename="$(find vetex_support)/urdf/vetex_macro.xacro" />
+<xacro:include filename="$(find euler_support)/urdf/asus_xtion_pro.xacro" />
         <xacro:macro name="euler" params="prefix">
         <xacro:vetex prefix="vetex_" />
         <xacro:motoman_mh5lf prefix="motoman_" />
+        <xacro:asus_xtion_pro sensor_name="" off_x="0.461" off_y="0" off_z="2.103" off_rr="1.5708" off_rp="1.8849" off_ry="0"/>
         <!--link list -->
-        <link name="base_link"> </link>
-        <link name="frame_left">
+        <link name="${prefix}base_link"> </link>
+        <link name="${prefix}frame_left">
                 <visual>
                         <origin xyz="0 0 0" rpy="0 0 0" />
-                                <geometry>
-                                        <mesh filename="package://euler_support/meshes/visual/frame_left.stl" />
-                                </geometry>
-                                <material name="">
-                                        <color rgba="0.752941176470588 0.752941176470588 0.752941176470588 1" />
-                                </material>
+                        <geometry>
+                                <mesh filename="package://euler_support/meshes/visual/frame_left.stl" />
+                        </geometry>
+                        <material name="">
+                                <color rgba="0.752941176470588 0.752941176470588 0.752941176470588 1" />
+                        </material>
                 </visual>
                 <collision>
@@ -25,13 +27,13 @@
                 </collision>
         </link>
-        <link name="frame_right">
+        <link name="${prefix}frame_right">
                 <visual>
                         <origin xyz="0 0 0" rpy="0 0 0" />
-                                <geometry>
-                                        <mesh filename="package://euler_support/meshes/visual/frame_right.stl" />
-                                </geometry>
-                                <material name="">
-                                        <color rgba="0.752941176470588 0.752941176470588 0.752941176470588 1" />
-                                </material>
+                        <geometry>
+                                <mesh filename="package://euler_support/meshes/visual/frame_right.stl" />
+                        </geometry>
+                        <material name="">
+                                <color rgba="0.752941176470588 0.752941176470588 0.752941176470588 1" />
+                        </material>
                 </visual>
                 <collision>
@@ -42,13 +44,13 @@
                 </collision>
         </link>
-        <link name="frame_top">
+        <link name="${prefix}frame_top">
                 <visual>
                         <origin xyz="0 0 0" rpy="0 0 0" />
-                                <geometry>
-                                        <mesh filename="package://euler_support/meshes/visual/frame_top.stl" />
-                                </geometry>
-                                <material name="">
-                                        <color rgba="0.752941176470588 0.752941176470588 0.752941176470588 1" />
-                                </material>
+                        <geometry>
+                                <mesh filename="package://euler_support/meshes/visual/frame_top.stl" />
+                        </geometry>
+                        <material name="">
+                                <color rgba="0.752941176470588 0.752941176470588 0.752941176470588 1" />
+                        </material>
                 </visual>
                 <collision>
@@ -59,32 +61,101 @@
                 </collision>
         </link>
-        <joint name="frame_left" type="fixed" >
-                <parent link="base_link" />
-                <child link="frame_left" />
+        <link name="${prefix}sick_nav350">
+                <visual>
+                        <origin xyz="-0.239 -0.648 2.551" rpy="0 0 0" />
+                        <geometry>
+                                <mesh filename="package://euler_support/meshes/visual/sick_nav350.stl" />
+                        </geometry>
+                        <material name="">
+                                <color rgba="0 0 0.752941176470588 1" />
+                        </material>
+                </visual>
+                <collision>
+                        <origin xyz="-0.239 -0.648 2.551" rpy="0 0 0" />
+                        <geometry>
+                                <mesh filename="package://euler_support/meshes/collision/sick_nav350.stl" />
+                        </geometry>
+                </collision>
+        </link>
+        <link name="${prefix}front_sick_s300">
+                <visual>
+                        <origin xyz="0.193 -0.617 0.532" rpy="0 0 -0.75047" />
+                        <geometry>
+                                <mesh filename="package://euler_support/meshes/visual/sick_s300_mounting_assy.stl" />
+                        </geometry>
+                        <material name="">
+                                <color rgba="0.75 0.75 0 1" />
+                        </material>
+                </visual>
+                <collision>
+                        <origin xyz="0.193 0.617 0.532" rpy="0 0 -0.75047" />
+                        <geometry>
+                                <mesh filename="package://euler_support/meshes/collision/sick_s300_mounting_assy.stl" />
+                        </geometry>
+                </collision>
+        </link>
+        <link name="${prefix}rear_sick_s300">
+                <visual>
+                        <origin xyz="-2.280 0.617 0.532" rpy="0 0  -3.96178" />
+                        <geometry>
+                                <mesh filename="package://euler_support/meshes/visual/sick_s300_mounting_assy.stl" />
+                        </geometry>
+                        <material name="">
+                                <color rgba="0.75 0.75 0 1" />
+                        </material>
+                </visual>
+                <collision>
+                        <origin xyz="-2.280 -0.617 0.532" rpy="0 0 -3.96178" />
+                        <geometry>
+                                <mesh filename="package://euler_support/meshes/collision/sick_s300_mounting_assy.stl" />
+                        </geometry>
+                </collision>
+        </link>
+        <joint name="${prefix}frame_left" type="fixed" >
+                <parent link="${prefix}base_link" />
+                <child link="${prefix}frame_left" />
                 <origin xyz="0 0 0" rpy="0 0 0" />
                 <axis xyz="0 0 0" />
         </joint>
-        <joint name="frame_right" type="fixed">
-                <parent link="base_link" />
-                <child link="frame_right" />
+        <joint name="${prefix}frame_right" type="fixed">
+                <parent link="${prefix}base_link" />
+                <child link="${prefix}frame_right" />
                 <origin xyz="0 0 0" rpy="0 0 0" />
                 <axis xyz="0 0 0" />
         </joint>
-        <joint name="frame_top" type="fixed">
-                <parent link="base_link" />
-                <child link="frame_top" />
+        <joint name="${prefix}frame_top" type="fixed">
+                <parent link="${prefix}base_link" />
+                <child link="${prefix}frame_top" />
                 <origin xyz="0 0 0" rpy="0 0 0" />
                 <axis xyz="0 0 0" />
         </joint>
-        <joint name="to_vetex" type="fixed">
-                <parent link="base_link" />
-                <child link="vetex_base_link" />
+        <joint name="${prefix}to_vetex" type="fixed">
+                <parent link="${prefix}base_link" />
+                <child link="${prefix}vetex_base_link" />
                 <origin xyz="0 0 0" rpy="0 0 0" />
                 <axis xyz="0 0 0" />
         </joint>
-        <joint name="to_arm" type="fixed">
-                <parent link="base_link" />
-                <child link="motoman_base_link" />
+        <joint name="${prefix}to_arm" type="fixed">
+                <parent link="${prefix}base_link" />
+                <child link="${prefix}motoman_base_link" />
                 <origin xyz="0.067518 0 2.016" rpy="3.1415 0 0" />
+                <axis xyz="0 0 0" />
+        </joint>
+        <joint name="${prefix}sick_nav350" type="fixed">
+                <parent link="${prefix}base_link" />
+                <child link="${prefix}sick_nav350" />
+                <origin xyz="0 0 0" rpy="0 0 0" />
+                <axis xyz="0 0 0" />
+        </joint>
+        <joint name="${prefix}front_sick_s300" type="fixed">
+                <parent link="${prefix}base_link" />
+                <child link="${prefix}front_sick_s300" />
+                <origin xyz="0 0 0" rpy="0 0 0" />
+                <axis xyz="0 0 0" />
+        </joint>
+                <joint name="${prefix}rear_sick_s300" type="fixed">
+                <parent link="${prefix}base_link" />
+                <child link="${prefix}rear_sick_s300" />
+                <origin xyz="0 0 0" rpy="0 0 0" />
                 <axis xyz="0 0 0" />
         </joint>

Commit message: Reverted vetex_bas_footprint to original orientation.  Vetex driver will be updated to match new orientation in subsequent commit

File: euler_support/urdf/euler.urdf (robot description, URDF)
Before this commit: robot euler, 24 links, 23 joints
Links:
- removed link vetex_map
- removed link vetex_odom
- added link eef_base
- added link eef_body; collision mesh filename=package://euler_support/meshes/collision/eef_vacuum.stl; visual mesh filename=package://euler_support/meshes/visual/eef_vacuum.stl
- added link localization_frame
- added link tcp
- added link vetex_base_footprint
Joints:
- removed joint vetex_map
- removed joint vetex_odom
- added joint base_to_localization: type fixed, parent base_link, child localization_frame, origin xyz=-0.239 -0.648 0 rpy=0 0 0, axis 0 0 0
- added joint eef_base_to_eef_body: type fixed, parent eef_base, child eef_body, origin xyz=0 0 0 rpy=0 0 1.57
- added joint eef_base_to_tcp: type fixed, parent eef_base, child tcp, origin xyz=0 0 0.17 rpy=0 0 0
- added joint motoman_link_t_to_eef_base: type fixed, parent motoman_link_t, child eef_base, origin xyz=0.098 0 0 rpy=0 1.57 0
- added joint vetex_to_footprint: type fixed, parent vetex_base_link, child vetex_base_footprint, origin xyz=-1.0439 0 0
- joint front_sick_s300: origin xyz=0 0 0 rpy=0 0 0 -> xyz=0.193 -0.617 0.532 rpy=0 0 -0.75047
- joint rear_sick_s300: origin xyz=0 0 0 rpy=0 0 0 -> xyz=-2.280 0.617 0.532 rpy=0 0  -3.96178
- joint sick_nav350: origin xyz=0 0 0 rpy=0 0 0 -> xyz=-0.239 -0.648 2.551 rpy=0 0 0
- joint vetex_left_front_wheel: limit lower=-10 upper=10 effort=0 velocity=3 -> effort=0 velocity=3; parent vetex_odom -> vetex_base_link; type revolute -> continuous
- joint vetex_left_rear_wheel: limit lower=-10 upper=10 effort=0 velocity=3 -> effort=0 velocity=3; parent vetex_odom -> vetex_base_link; type revolute -> continuous
- joint vetex_right_front_wheel: limit lower=-10 upper=10 effort=0 velocity=3 -> effort=0 velocity=3; parent vetex_odom -> vetex_base_link; type revolute -> continuous
- joint vetex_right_rear_wheel: limit lower=-10 upper=10 effort=0 velocity=3 -> effort=0 velocity=3; parent vetex_odom -> vetex_base_link; type revolute -> continuous

File: vetex_support/urdf/vetex_macro.xacro (robot description, xacro)
@@ -78,5 +78,5 @@
                 <!-- joint list -->
                 <joint name="${prefix}to_footprint" type="fixed">
-                    <origin xyz="-1.0439 0 0" rpy="0 0 1.57"/>
+                    <origin xyz="-1.0439 0 0" />
                     <parent link="${prefix}base_link" />
                     <child link="${prefix}base_footprint" />
