Commit message: moved robot back in to euler_macro.xacro, cleaned bugs

File: euler_support/urdf/asus_xtion_pro.xacro (robot description, xacro)
@@ -20,21 +20,21 @@
     </collision>
   </link>
-  <joint name="${sensor_name}_base-bodycenter-prism-x" type="fixed">
+  <joint name="${sensor_name}base-bodycenter-prism-x" type="fixed">
     <origin xyz="${off_x} ${off_y} ${off_z}" rpy="${off_rr} ${off_rp} ${off_ry}" />
     <parent link="base_link" />
-    <child link="${sensor_name}_bodycenter" />
+    <child link="${sensor_name}bodycenter" />
   </joint>
-  <joint name="${sensor_name}_depth_joint" type="fixed">
+  <joint name="${sensor_name}depth_joint" type="fixed">
     <origin xyz="0.049 0 0" rpy="0 0 0" />
-    <parent link="${sensor_name}_bodycenter" />
-    <child link="${sensor_name}_depth_frame" />
+    <parent link="${sensor_name}bodycenter" />
+    <child link="${sensor_name}depth_frame" />
   </joint>
-  <link name="${sensor_name}_depth_frame" />
-  <joint name="${sensor_name}_rgb_joint" type="fixed">
+  <link name="${sensor_name}depth_frame" />
+  <joint name="${sensor_name}rgb_joint" type="fixed">
     <origin xyz="0.022 0 0" rpy="0 0 0" />
-    <parent link="${sensor_name}_bodycenter" />
-    <child link="${sensor_name}_rgb_frame" />
+    <parent link="${sensor_name}bodycenter" />
+    <child link="${sensor_name}rgb_frame" />
   </joint>
-  <link name="${sensor_name}_rgb_frame" />
+  <link name="${sensor_name}rgb_frame" />
 </xacro:macro>
 </robot>

File: euler_support/urdf/eef_macro.xacro (robot description, xacro)
@@ -10,5 +10,5 @@
           <origin xyz="0 0 0" rpy="0 0 0" />
           <geometry>
-                  <mesh filename="package://euler_support/meshes/visual/motoman_eef.stl" />
+                  <mesh filename="package://euler_support/meshes/visual/vacuum_gripper.stl" />
           </geometry>
           <material name="eef_color"/>
@@ -17,5 +17,5 @@
           <origin xyz="0 0 0" rpy="0 0 0" />
           <geometry>
-                  <mesh filename="package://euler_support/meshes/collision/motoman_eef.stl" />
+                  <mesh filename="package://euler_support/meshes/collision/vacuum_gripper.stl" />
           </geometry>
           <material name="eef_color"/>

File: euler_support/urdf/euler.xacro (robot description, xacro)
@@ -1,24 +1,5 @@
 <?xml version="1.0" ?>
 <robot name="euler" xmlns:xacro="http://ros.org/wiki/xacro">
-    <xacro:include filename="$(find motoman_mh5lf_support)/urdf/mh5lf_macro.xacro" />
-    <xacro:motoman_mh5lf prefix="motoman_" />
-    <xacro:include filename="$(find industrial_extrinsic_cal)/urdf/asus_sensor_cal_macro.xacro" />
-    <xacro:asus_sensor_definitions prefix="asus" parent_link="motoman_base_link" />
-    <xacro:include filename="$(find euler_support)/urdf/eef_macro.xacro"/>
-    <xacro:eef prefix=""/>
     <xacro:include filename="$(find euler_support)/urdf/euler_macro.xacro" />
     <xacro:euler prefix="euler_"/>
-    <!--euler to motoman link-->
-    <joint name="euler_to_arm" type="fixed">
-        <parent link="euler_base_link" />
-        <child link="motoman_base_link" />
-        <origin xyz="0.067518 0 2.016" rpy="3.1415 0 0" />
-        <axis xyz="0 0 0" />
-    </joint>
-    <!--motoman to end effector link-->
-    <joint name="motoman_link_t_to_eef_base" type="fixed">
-      <parent link="motoman_link_t" />
-      <child link="eef_base" />
-      <origin xyz="0.098 0 0" rpy="0 1.57 0" />
-    </joint>
 </robot>

File: euler_support/urdf/euler_macro.xacro (robot description, xacro)
@@ -1,6 +1,13 @@
 <?xml version="1.0" ?>
 <robot xmlns:xacro="http://ros.org/wiki/xacro">
-<xacro:include filename="$(find vetex_support)/urdf/vetex_macro.xacro" />
-        <xacro:macro name="euler" params="prefix">
+    <xacro:macro name="euler" params="prefix">
+        <xacro:include filename="$(find motoman_mh5lf_support)/urdf/mh5lf_macro.xacro" />
+        <xacro:motoman_mh5lf prefix="${prefix}motoman_" />
+        <!--xacro:include filename="$(find euler_support)/urdf/asus_xtion_pro.xacro" /-->
+        <xacro:include filename="$(find industrial_extrinsic_cal)/urdf/asus_sensor_cal_macro.xacro" />
+        <xacro:asus_sensor_definitions prefix="${prefix}asus_" parent_link="euler_motoman_base_link" />
+        <xacro:include filename="$(find euler_support)/urdf/eef_macro.xacro"/>
+        <xacro:eef prefix="${prefix}eef_"/>
+        <xacro:include filename="$(find vetex_support)/urdf/vetex_macro.xacro" />
         <xacro:vetex prefix="${prefix}vetex_" />
         <!--link list -->
@@ -151,4 +158,17 @@
                 <axis xyz="0 0 0" />
         </joint>
+        <!--euler to motoman link-->
+        <joint name="${prefix}platform_to_arm" type="fixed">
+            <parent link="${prefix}base_link" />
+            <child link="${prefix}motoman_base_link" />
+            <origin xyz="0.067518 0 2.016" rpy="3.1415 0 0" />
+            <axis xyz="0 0 0" />
+        </joint>
+        <!--motoman to end effector link-->
+        <joint name="${prefix}motoman_link_t_to_eef_base" type="fixed">
+          <parent link="${prefix}motoman_link_t" />
+          <child link="${prefix}eef_eef_base" />
+          <origin xyz="0.098 0 0" rpy="0 1.57 0" />
+        </joint>
 </xacro:macro>
 </robot>
