Commit message: Reposition origin of laser meshes

File: euler_support/urdf/euler_macro.xacro (robot description, xacro)
@@ -80,5 +80,4 @@
         <link name="${prefix}front_sick_s300">
                 <visual>
-                        <origin xyz="0.193 -0.617 0.532" rpy="0 0 -0.75047" />
                         <geometry>
                                 <mesh filename="package://euler_support/meshes/visual/sick_s300_mounting_assy.stl" />
@@ -89,5 +88,4 @@
                 </visual>
                 <collision>
-                        <origin xyz="0.193 0.617 0.532" rpy="0 0 -0.75047" />
                         <geometry>
                                 <mesh filename="package://euler_support/meshes/collision/sick_s300_mounting_assy.stl" />
@@ -97,5 +95,4 @@
         <link name="${prefix}rear_sick_s300">
                 <visual>
-                        <origin xyz="-2.280 0.617 0.532" rpy="0 0  -3.96178" />
                         <geometry>
                                 <mesh filename="package://euler_support/meshes/visual/sick_s300_mounting_assy.stl" />
@@ -106,5 +103,4 @@
                 </visual>
                 <collision>
-                        <origin xyz="-2.280 -0.617 0.532" rpy="0 0 -3.96178" />
                         <geometry>
                                 <mesh filename="package://euler_support/meshes/collision/sick_s300_mounting_assy.stl" />
@@ -151,5 +147,5 @@
                 <parent link="${prefix}base_link" />
                 <child link="${prefix}front_sick_s300" />
-                <origin xyz="0 0 0" rpy="0 0 0" />
+                <origin xyz="0.193 -0.617 0.532" rpy="0 0 -0.75047" />
                 <axis xyz="0 0 0" />
         </joint>
@@ -157,5 +153,5 @@
                 <parent link="${prefix}base_link" />
                 <child link="${prefix}rear_sick_s300" />
-                <origin xyz="0 0 0" rpy="0 0 0" />
+                <origin xyz="-2.280 0.617 0.532" rpy="0 0  -3.96178" />
                 <axis xyz="0 0 0" />
         </joint>

Commit message: added end effector to model

File: euler_support/urdf/euler_macro.xacro (robot description, xacro)
@@ -4,8 +4,10 @@
 <xacro:include filename="$(find motoman_mh5lf_support)/urdf/mh5lf_macro.xacro" />
 <xacro:include filename="$(find euler_support)/urdf/asus_xtion_pro.xacro" />
+<xacro:include filename="$(find euler_support)/urdf/eef_macro.xacro" />
         <xacro:macro name="euler" params="prefix">
         <xacro:vetex prefix="vetex_" />
         <xacro:motoman_mh5lf prefix="motoman_" />
         <xacro:asus_xtion_pro sensor_name="" off_x="0.461" off_y="0" off_z="2.103" off_rr="1.5708" off_rp="1.8849" off_ry="0"/>
+        <xacro:eef prefix=""/>
         <!--link list -->
         <link name="${prefix}base_link"> </link>
@@ -150,5 +152,5 @@
                 <axis xyz="0 0 0" />
         </joint>
-                <joint name="${prefix}rear_sick_s300" type="fixed">
+        <joint name="${prefix}rear_sick_s300" type="fixed">
                 <parent link="${prefix}base_link" />
                 <child link="${prefix}rear_sick_s300" />
@@ -156,4 +158,9 @@
                 <axis xyz="0 0 0" />
         </joint>
+        <joint name="motoman_link_t_to_eef_base" type="fixed">
+                <parent link="motoman_link_t" />
+                <child link="eef_base" />
+                <origin xyz="0.098 0 0" rpy="0 1.57 0" />
+        </joint>
 </xacro:macro>
 </robot>

Commit message: corrected frame location for sick_nav350 sensor

File: euler_support/urdf/euler_macro.xacro (robot description, xacro)
@@ -65,5 +65,4 @@
         <link name="${prefix}sick_nav350">
                 <visual>
-                        <origin xyz="-0.239 -0.648 2.551" rpy="0 0 0" />
                         <geometry>
                                 <mesh filename="package://euler_support/meshes/visual/sick_nav350.stl" />
@@ -74,5 +73,4 @@
                 </visual>
                 <collision>
-                        <origin xyz="-0.239 -0.648 2.551" rpy="0 0 0" />
                         <geometry>
                                 <mesh filename="package://euler_support/meshes/collision/sick_nav350.stl" />
@@ -143,5 +141,5 @@
                 <parent link="${prefix}base_link" />
                 <child link="${prefix}sick_nav350" />
-                <origin xyz="0 0 0" rpy="0 0 0" />
+                <origin xyz="-0.239 -0.648 2.551" rpy="0 0 0" />
                 <axis xyz="0 0 0" />
         </joint>

Commit message: created localization link at the bottom of the robot base

File: euler_support/urdf/euler_macro.xacro (robot description, xacro)
@@ -12,4 +12,5 @@
         <!--link list -->
         <link name="${prefix}base_link"> </link>
+	<link name="${prefix}localization_frame"/>
         <link name="${prefix}frame_left">
                 <visual>
@@ -144,4 +145,10 @@
                 <axis xyz="0 0 0" />
         </joint>
+        <joint name="${prefix}base_to_localization" type="fixed">
+                <parent link="${prefix}base_link" />
+                <child link="${prefix}localization_frame" />
+                <origin xyz="-0.239 -0.648 0" rpy="0 0 0" />
+                <axis xyz="0 0 0" />
+        </joint>
         <joint name="${prefix}front_sick_s300" type="fixed">
                 <parent link="${prefix}base_link" />

Commit message: added software robot base link and added calibration target links

File: euler_support/urdf/euler_macro.xacro (robot description, xacro)
@@ -14,5 +14,7 @@
         <!--link list -->
         <link name="${prefix}base_link"> </link>
-	<link name="${prefix}localization_frame"/>
+	      <link name="${prefix}localization_frame"/>
+	      <link name="calibration_target1"/>
+	      <link name="calibration_target2"/>
         <link name="${prefix}frame_left">
                 <visual>
@@ -170,4 +172,14 @@
                 <origin xyz="0.098 0 0" rpy="0 1.57 0" />
         </joint>
+        <joint name="motoman_base_to_cal_target1" type="fixed">
+                <parent link="motoman_base_link" />
+                <child link="calibration_target1" />
+                <origin xyz="0.4 0 0.7" rpy="3.1416 0 0" />
+        </joint>
+        <joint name="motoman_base_to_cal_target2" type="fixed">
+                <parent link="motoman_base_link" />
+                <child link="calibration_target2" />
+                <origin xyz="0.3 0 1.2" rpy="3.1416 0 0" />
+        </joint>
 </xacro:macro>
 </robot>

File: motoman_mh5lf_support/urdf/mh5lf_macro.xacro (robot description, xacro)
@@ -1,6 +1,8 @@
 <?xml version="1.0" ?>
 <robot xmlns:xacro="http://ros.org/wiki/xacro">
+	<xacro:property name="base_offset" value="0.330"/>
 	<xacro:macro name="motoman_mh5lf" params="prefix">
 		<!-- link list -->
+		<link name="${prefix}base_software"/>
 		<link name="${prefix}base_link">
 			<visual>
@@ -118,4 +120,9 @@
 			 <limit lower="-2.96697222222222" upper="2.96697222222222" effort="100" velocity="4.71225" />
 		</joint>
+		<joint name="${prefix}base_to_base_software" type="fixed">
+			<parent link="${prefix}base_link"/>
+			<child link="${prefix}base_software"/>
+			<origin xyz="0 0 ${base_offset}" rpy="0 0 0"/>
+		</joint>
 		<joint name="${prefix}joint_l" type="revolute">
 			<parent link="${prefix}link_s"/>

Commit message: tweeked mutable joints for camera

File: euler_support/urdf/euler_macro.xacro (robot description, xacro)
@@ -175,10 +175,10 @@
                 <parent link="motoman_base_link" />
                 <child link="calibration_target1" />
-                <origin xyz="0.4 0 0.7" rpy="3.1416 0 0" />
+                <origin xyz="0.7 -0.14 0.7" rpy="3.1416 0 0" />
         </joint>
         <joint name="motoman_base_to_cal_target2" type="fixed">
                 <parent link="motoman_base_link" />
                 <child link="calibration_target2" />
-                <origin xyz="0.3 0 1.2" rpy="3.1416 0 0" />
+                <origin xyz="0.4 0.0 1.2" rpy="3.1416 0 0" />
         </joint>
 </xacro:macro>

Commit message: removed calibration target links and joints

File: euler_support/urdf/euler_macro.xacro (robot description, xacro)
@@ -15,6 +15,4 @@
         <link name="${prefix}base_link"> </link>
 	      <link name="${prefix}localization_frame"/>
-	      <link name="calibration_target1"/>
-	      <link name="calibration_target2"/>
         <link name="${prefix}frame_left">
                 <visual>
@@ -172,14 +170,4 @@
                 <origin xyz="0.098 0 0" rpy="0 1.57 0" />
         </joint>
-        <joint name="motoman_base_to_cal_target1" type="fixed">
-                <parent link="motoman_base_link" />
-                <child link="calibration_target1" />
-                <origin xyz="0.7 -0.14 0.7" rpy="3.1416 0 0" />
-        </joint>
-        <joint name="motoman_base_to_cal_target2" type="fixed">
-                <parent link="motoman_base_link" />
-                <child link="calibration_target2" />
-                <origin xyz="0.4 0.0 1.2" rpy="3.1416 0 0" />
-        </joint>
 </xacro:macro>
 </robot>

Commit message: updated dependencies and old references

File: euler_support/urdf/euler_macro.xacro (robot description, xacro)
@@ -11,5 +11,5 @@
         <!--xacro:asus_xtion_pro sensor_name="" off_x="0.461" off_y="0" off_z="2.103" off_rr="1.5708" off_rp="1.8849" off_ry="0"/-->
         <xacro:asus_sensor_definitions prefix="asus" parent_link="motoman_base_link" />
-        <xacro:eef prefix=""/>
+        <!--<xacro:eef prefix=""/>-->
         <!--link list -->
         <link name="${prefix}base_link"> </link>
@@ -165,9 +165,9 @@
                 <axis xyz="0 0 0" />
         </joint>
-        <joint name="motoman_link_t_to_eef_base" type="fixed">
+        <!--<joint name="motoman_link_t_to_eef_base" type="fixed">
                 <parent link="motoman_link_t" />
                 <child link="eef_base" />
                 <origin xyz="0.098 0 0" rpy="0 1.57 0" />
-        </joint>
+        </joint>-->
 </xacro:macro>
 </robot>
