Commit message: added new end effector, cleaned macro references

File: euler_support/urdf/eef_macro.xacro (robot description, xacro)
@@ -2,5 +2,5 @@
 <robot xmlns:xacro="http://ros.org/wiki/xacro">
   <xacro:macro name="eef" params="prefix">
-    <material name="eef_color">
+    <material name="${prefix}eef_color">
             <color rgba="0.5 0.5 0.5 1" />
     </material>
@@ -10,5 +10,5 @@
           <origin xyz="0 0 0" rpy="0 0 0" />
           <geometry>
-                  <mesh filename="package://euler_support/meshes/visual/eef_vacuum.stl" />
+                  <mesh filename="package://euler_support/meshes/visual/motoman_eef.stl" />
           </geometry>
           <material name="eef_color"/>
@@ -17,5 +17,5 @@
           <origin xyz="0 0 0" rpy="0 0 0" />
           <geometry>
-                  <mesh filename="package://euler_support/meshes/collision/eef_vacuum.stl" />
+                  <mesh filename="package://euler_support/meshes/collision/motoman_eef.stl" />
           </geometry>
           <material name="eef_color"/>
@@ -26,5 +26,5 @@
       <parent link="${prefix}eef_base" />
       <child link="${prefix}eef_body" />
-      <origin xyz="0 0 0" rpy="0 0 1.57" />
+      <origin xyz="0 0 0" rpy="-1.57 0 1.57" />
     </joint>
     <joint name="${prefix}eef_base_to_${prefix}tcp" type="fixed">

File: euler_support/urdf/euler.xacro (robot description, xacro)
@@ -1,5 +1,24 @@
 <?xml version="1.0" ?>
 <robot name="euler" xmlns:xacro="http://ros.org/wiki/xacro">
-        <xacro:include filename="$(find euler_support)/urdf/euler_macro.xacro" />
-        <xacro:euler prefix=""/>
+    <xacro:include filename="$(find motoman_mh5lf_support)/urdf/mh5lf_macro.xacro" />
+    <xacro:motoman_mh5lf prefix="motoman_" />
+    <xacro:include filename="$(find industrial_extrinsic_cal)/urdf/asus_sensor_cal_macro.xacro" />
+    <xacro:asus_sensor_definitions prefix="asus" parent_link="motoman_base_link" />
+    <xacro:include filename="$(find euler_support)/urdf/eef_macro.xacro"/>
+    <xacro:eef prefix=""/>
+    <xacro:include filename="$(find euler_support)/urdf/euler_macro.xacro" />
+    <xacro:euler prefix="euler_"/>
+    <!--euler to motoman link-->
+    <joint name="euler_to_arm" type="fixed">
+        <parent link="euler_base_link" />
+        <child link="motoman_base_link" />
+        <origin xyz="0.067518 0 2.016" rpy="3.1415 0 0" />
+        <axis xyz="0 0 0" />
+    </joint>
+    <!--motoman to end effector link-->
+    <joint name="motoman_link_t_to_eef_base" type="fixed">
+      <parent link="motoman_link_t" />
+      <child link="eef_base" />
+      <origin xyz="0.098 0 0" rpy="0 1.57 0" />
+    </joint>
 </robot>

File: euler_support/urdf/euler_macro.xacro (robot description, xacro)
@@ -2,14 +2,6 @@
 <robot xmlns:xacro="http://ros.org/wiki/xacro">
 <xacro:include filename="$(find vetex_support)/urdf/vetex_macro.xacro" />
-<xacro:include filename="$(find motoman_mh5lf_support)/urdf/mh5lf_macro.xacro" />
-<!--xacro:include filename="$(find euler_support)/urdf/asus_xtion_pro.xacro" /-->
-<xacro:include filename="$(find industrial_extrinsic_cal)/urdf/asus_sensor_cal_macro.xacro" />
-<xacro:include filename="$(find euler_support)/urdf/eef_macro.xacro" />
         <xacro:macro name="euler" params="prefix">
-        <xacro:vetex prefix="vetex_" />
-        <xacro:motoman_mh5lf prefix="motoman_" />
-        <!--xacro:asus_xtion_pro sensor_name="" off_x="0.461" off_y="0" off_z="2.103" off_rr="1.5708" off_rp="1.8849" off_ry="0"/-->
-        <xacro:asus_sensor_definitions prefix="asus" parent_link="motoman_base_link" />
-        <!--<xacro:eef prefix=""/>-->
+        <xacro:vetex prefix="${prefix}vetex_" />
         <!--link list -->
         <link name="${prefix}base_link"> </link>
@@ -135,10 +127,4 @@
                 <axis xyz="0 0 0" />
         </joint>
-        <joint name="${prefix}to_arm" type="fixed">
-                <parent link="${prefix}base_link" />
-                <child link="${prefix}motoman_base_link" />
-                <origin xyz="0.067518 0 2.016" rpy="3.1415 0 0" />
-                <axis xyz="0 0 0" />
-        </joint>
         <joint name="${prefix}sick_nav350" type="fixed">
                 <parent link="${prefix}base_link" />
@@ -165,9 +151,4 @@
                 <axis xyz="0 0 0" />
         </joint>
-        <!--<joint name="motoman_link_t_to_eef_base" type="fixed">
-                <parent link="motoman_link_t" />
-                <child link="eef_base" />
-                <origin xyz="0.098 0 0" rpy="0 1.57 0" />
-        </joint>-->
 </xacro:macro>
 </robot>

File: motoman_mh5lf_support/urdf/mh5lf_macro.xacro (robot description, xacro)
@@ -2,5 +2,5 @@
 <robot xmlns:xacro="http://ros.org/wiki/xacro">
 	<xacro:property name="base_offset" value="0.330"/>
-	<xacro:macro name="motoman_mh5lf" params="prefix">
+        <xacro:macro name="motoman_mh5lf" params="prefix">
 		<!-- link list -->
 		<link name="${prefix}base_software"/>

Commit message: Fixes to colors in eef macro

File: euler_support/urdf/eef_macro.xacro (robot description, xacro)
@@ -3,5 +3,5 @@
   <xacro:macro name="eef" params="prefix">
     <material name="${prefix}eef_color">
-            <color rgba="0.5 0.5 0.5 1" />
+      <color rgba="0.5 0.5 0.5 1" />
     </material>
     <link name="${prefix}eef_base"/>
@@ -12,5 +12,5 @@
           <mesh filename="package://euler_support/meshes/visual/vacuum_gripper.stl" />
         </geometry>
-        <material name="eef_color"/>
+        <material name="${prefix}eef_color"/>
       </visual>
       <collision>
@@ -19,5 +19,5 @@
           <mesh filename="package://euler_support/meshes/collision/vacuum_gripper.stl" />
         </geometry>
-        <material name="eef_color"/>
+        <material name="${prefix}eef_color"/>
       </collision>
     </link>

Commit message: Updated TCP location

File: euler_support/urdf/eef_macro.xacro (robot description, xacro)
@@ -26,10 +26,10 @@
       <parent link="${prefix}eef_base" />
       <child link="${prefix}eef_body" />
-      <origin xyz="0 0 0" rpy="-1.57 0 1.57" />
+      <origin xyz="0 0 0" rpy="-${radians(90)} 0 ${radians(90)}" />
     </joint>
     <joint name="${prefix}eef_base_to_${prefix}tcp" type="fixed">
       <parent link="${prefix}eef_base" />
       <child link="${prefix}tcp" />
-      <origin xyz="0 0 0.17" rpy="0 0 0" />
+      <origin xyz="0 0 0.085" rpy="0 0 0" />
     </joint>
   </xacro:macro>

Commit message: Updated eef macro link naming

File: euler_support/urdf/eef_macro.xacro (robot description, xacro)
@@ -2,9 +2,9 @@
 <robot xmlns:xacro="http://ros.org/wiki/xacro">
   <xacro:macro name="eef" params="prefix">
-    <material name="${prefix}eef_color">
+    <material name="${prefix}color">
       <color rgba="0.5 0.5 0.5 1" />
     </material>
-    <link name="${prefix}eef_base"/>
-    <link name="${prefix}eef_body">
+    <link name="${prefix}base_link"/>
+    <link name="${prefix}body">
       <visual>
         <origin xyz="0 0 0" rpy="0 0 0" />
@@ -12,5 +12,5 @@
           <mesh filename="package://euler_support/meshes/visual/vacuum_gripper.stl" />
         </geometry>
-        <material name="${prefix}eef_color"/>
+        <material name="${prefix}color"/>
       </visual>
       <collision>
@@ -19,15 +19,15 @@
           <mesh filename="package://euler_support/meshes/collision/vacuum_gripper.stl" />
         </geometry>
-        <material name="${prefix}eef_color"/>
+        <material name="${prefix}color"/>
       </collision>
     </link>
     <link name="${prefix}tcp"/>
-    <joint name="${prefix}eef_base_to_${prefix}eef_body" type="fixed">
-      <parent link="${prefix}eef_base" />
-      <child link="${prefix}eef_body" />
+    <joint name="${prefix}body_to_base_link" type="fixed">
+      <parent link="${prefix}base_link" />
+      <child link="${prefix}body" />
       <origin xyz="0 0 0" rpy="-${radians(90)} 0 ${radians(90)}" />
     </joint>
-    <joint name="${prefix}eef_base_to_${prefix}tcp" type="fixed">
-      <parent link="${prefix}eef_base" />
+    <joint name="${prefix}tcp_to_base_link" type="fixed">
+      <parent link="${prefix}base_link" />
       <child link="${prefix}tcp" />
       <origin xyz="0 0 0.085" rpy="0 0 0" />

File: euler_support/urdf/euler_macro.xacro (robot description, xacro)
@@ -10,6 +10,7 @@
     <xacro:asus_sensor_definitions prefix="${prefix}asus" parent_link="${robot_prefix}base_link"/>
     <!-- End effector -->
+    <xacro:property name="eef_prefix" value="eef_"/>
     <xacro:include filename="$(find euler_support)/urdf/eef_macro.xacro"/>
-    <xacro:eef prefix="${prefix}eef_"/>
+    <xacro:eef prefix="${prefix+eef_prefix}"/>
     <!-- Mobile Platform -->
     <xacro:include filename="$(find vetex_support)/urdf/vetex_macro.xacro"/>
@@ -170,7 +171,7 @@
     </joint>
     <!--motoman to end effector link-->
-    <joint name="${prefix+robot_prefix}link_t_to_eef_base" type="fixed">
+    <joint name="${prefix+robot_prefix}link_t_to_${eef_prefix}base_link" type="fixed">
       <parent link="${prefix+robot_prefix}link_t"/>
-      <child link="${prefix}eef_eef_base"/>
+      <child link="${prefix+eef_prefix}base_link"/>
       <origin xyz="0.098 0 0" rpy="0 1.57 0"/>
     </joint>
